Commit message: Add modified urdf

File: ur_description/urdf/ur5_joint_limited.urdf.xacro (robot description, xacro)
@@ -43,4 +43,5 @@
   <property name="forearm_radius" value="0.040" />    <!-- manually measured -->
   <property name="wrist_radius" value="0.045" />      <!-- manually measured -->
+  <property name="damping" value="5.0" />
 <xacro:macro name="ur5_robot" params="prefix">
   <link name="${prefix}base_link" >
@@ -59,5 +60,5 @@
     <inertial>
       <mass value="${base_mass}" />
-      <inertia ixx="1.0" ixy="0.0" ixz="0.0" iyy="1.0" iyz="0.0" izz="1.0"/>
+      <inertia ixx="0.002" ixy="0.0" ixz="0.0" iyy="0.02" iyz="0.0" izz="0.002"/>
     </inertial>
   </link>
@@ -68,5 +69,5 @@
     <axis xyz="0 0 1" />
     <limit lower="${-pi}" upper="${pi}" effort="150.0" velocity="${pi}"/>
-    <dynamics damping="0.4" friction="0.0"/>
+    <dynamics damping="${damping}" friction="0.0"/>
   </joint>
   <link name="${prefix}shoulder_link">
@@ -84,5 +85,5 @@
     <inertial>
       <mass value="${shoulder_mass}" />
-      <inertia ixx="1.0" ixy="0.0" ixz="0.0" iyy="1.0" iyz="0.0" izz="1.0"/>
+      <inertia ixx="0.002" ixy="0.0" ixz="0.0" iyy="0.02" iyz="0.0" izz="0.002"/>
       <origin xyz="${shoulder_cog}" rpy="0.0 0.0 0.0" />
     </inertial>
@@ -94,5 +95,5 @@
     <axis xyz="0 1 0" />
     <limit lower="${-pi}" upper="${pi}" effort="150.0" velocity="${pi}"/>
-    <dynamics damping="0.4" friction="0.0"/>
+    <dynamics damping="${damping}" friction="0.0"/>
   </joint>
   <link name="${prefix}upper_arm_link">
@@ -111,5 +112,5 @@
     <inertial>
       <mass value="${upper_arm_mass}" />
-      <inertia ixx="1.0" ixy="0.0" ixz="0.0" iyy="1.0" iyz="0.0" izz="1.0"/>
+      <inertia ixx="0.002" ixy="0.0" ixz="0.0" iyy="0.02" iyz="0.0" izz="0.002"/>
       <origin xyz="${upper_arm_cog}" rpy="0.0 0.0 0.0" />
     </inertial>
@@ -121,5 +122,5 @@
     <axis xyz="0 1 0" />
     <limit lower="${-pi}" upper="${pi}" effort="150.0" velocity="${pi}"/>
-    <dynamics damping="0.4" friction="0.0"/>
+    <dynamics damping="${damping}" friction="0.0"/>
   </joint>
   <link name="${prefix}forearm_link">
@@ -138,5 +139,5 @@
       <mass value="${forearm_mass}" />
       <origin xyz="${forearm_cog}" rpy="0.0 0.0 0.0" />
-      <inertia ixx="1.0" ixy="0.0" ixz="0.0" iyy="1.0" iyz="0.0" izz="1.0"/>
+      <inertia ixx="0.002" ixy="0.0" ixz="0.0" iyy="0.02" iyz="0.0" izz="0.002"/>
     </inertial>
   </link>
@@ -147,5 +148,5 @@
     <axis xyz="0 1 0" />
     <limit lower="${-1.0 * pi}" upper="${0.25 * pi}" effort="28.0" velocity="${pi}"/>
-    <dynamics damping="0.3" friction="0.0"/>
+    <dynamics damping="${damping}" friction="0.0"/>
   </joint>
   <link name="${prefix}wrist_1_link">
@@ -165,5 +166,5 @@
       <mass value="${wrist_1_mass}" />
       <origin xyz="${wrist_1_cog}" rpy="0.0 0.0 0.0" />
-      <inertia ixx="1.0" ixy="0.0" ixz="0.0" iyy="1.0" iyz="0.0" izz="1.0"/>
+      <inertia ixx="0.002" ixy="0.0" ixz="0.0" iyy="0.02" iyz="0.0" izz="0.002"/>
     </inertial>
   </link>
@@ -174,5 +175,5 @@
     <axis xyz="0 0 1" />
     <limit lower="${-1.0 * pi}" upper="${1.0 * pi}" effort="28.0" velocity="${pi}"/>
-    <dynamics damping="0.3" friction="0.0"/>
+    <dynamics damping="${damping}" friction="0.0"/>
   </joint>
   <link name="${prefix}wrist_2_link">
@@ -192,5 +193,5 @@
       <mass value="${wrist_2_mass}" />
       <origin xyz="${wrist_2_cog}" rpy="0.0 0.0 0.0" />
-      <inertia ixx="1.0" ixy="0.0" ixz="0.0" iyy="1.0" iyz="0.0" izz="1.0"/>
+      <inertia ixx="0.002" ixy="0.0" ixz="0.0" iyy="0.02" iyz="0.0" izz="0.002"/>
     </inertial>
   </link>
@@ -201,5 +202,5 @@
     <axis xyz="0 1 0" />
     <limit lower="${-1.0 * pi}" upper="${1.0 * pi}" effort="28.0" velocity="${pi}"/>
-    <dynamics damping="0.3" friction="0.0"/>
+    <dynamics damping="${damping}" friction="0.0"/>
   </joint>
   <link name="${prefix}wrist_3_link">
@@ -217,5 +218,5 @@
       <mass value="${wrist_3_mass}" />
       <origin xyz="${wrist_3_cog}" rpy="0.0 0.0 0.0" />
-      <inertia ixx="1.0" ixy="0.0" ixz="0.0" iyy="1.0" iyz="0.0" izz="1.0"/>
+      <inertia ixx="0.002" ixy="0.0" ixz="0.0" iyy="0.02" iyz="0.0" izz="0.002"/>
     </inertial>
   </link>
